File: 01-getting-started/01-getting-started/01-getting-started.kicad_sch (KiCad schematic)
At the start: 3 parts

Commit message: Add finished project
Parts:
- added SW1: M2011S3A1W03, getting-started:Switch_Toggle_SPST_NKK_M2011S3A1x03, symbol getting-started:M2011S3A1W03
Connections:
- net VCC: now also SW1.3 (B); no longer BT1.1 (+)
- new net: BT1.1 (+), SW1.2 (A)
Other:
- moved on the sheet: BT1
Changed lines of the file:
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@@
     (rev "0")
-  )
-  (junction (at 119.38 77.47) (diameter 0) (color 0 0 0 0)
   )
   (junction (at 143.51 115.57) (diameter 0) (color 0 0 0 0)
@@
   (junction (at 143.51 68.58) (diameter 0) (color 0 0 0 0)
   )
-  (wire (pts (xy 119.38 77.47) (xy 119.38 87.63))
-    (stroke (width 0) (type default))
+  (junction (at 119.38 72.39) (diameter 0) (color 0 0 0 0)
   )
   (wire (pts (xy 167.64 83.82) (xy 167.64 100.33))
@@
     (stroke (width 0) (type default))
   )
-  (wire (pts (xy 119.38 77.47) (xy 119.38 68.58))
+  (wire (pts (xy 119.38 72.39) (xy 119.38 80.01))
     (stroke (width 0) (type default))
   )
@@
     (stroke (width 0) (type default))
   )
-  (wire (pts (xy 119.38 95.25) (xy 119.38 102.87))
+  (wire (pts (xy 119.38 99.06) (xy 119.38 102.87))
     (stroke (width 0) (type default))
   )
@@
     (stroke (width 0) (type default))
   )
+  (wire (pts (xy 119.38 90.17) (xy 119.38 91.44))
+    (stroke (width 0) (type default))
+  )
+  (wire (pts (xy 119.38 72.39) (xy 119.38 68.58))
+    (stroke (width 0) (type default))
+  )
   (wire (pts (xy 143.51 68.58) (xy 167.64 68.58))
     (stroke (width 0) (type default))
@@
     (effects (font (size 1.27 1.27)) (justify left bottom))
   )
-  (symbol (lib_id "power:PWR_FLAG") (at 119.38 77.47 90) (unit 1)
-    (in_bom yes) (on_board yes) (dnp no)
-    (property "Reference" "#FLG01" (at 117.475 77.47 0)
+  (symbol (lib_id "getting-started:M2011S3A1W03") (at 119.38 85.09 90) (unit 1)
+    (in_bom yes) (on_board yes) (dnp no) (fields_autoplaced)
+    (property "Reference" "SW1" (at 120.65 82.7088 90)
+      (effects (font (size 1.27 1.27)) (justify right))
+    )
+    (property "Value" "M2011S3A1W03" (at 120.65 85.2488 90)
+      (effects (font (size 1.27 1.27)) (justify right))
+    )
+    (property "Footprint" "getting-started:Switch_Toggle_SPST_NKK_M2011S3A1x03" (at 119.38 85.09 0)
       (effects (font (size 1.27 1.27)) hide)
     )
-    (property "Value" "PWR_FLAG" (at 114.3 77.47 0)
+    (property "Datasheet" "" (at 119.38 85.09 0)
+      (effects (font (size 1.27 1.27)) hide)
+    )
+    (pin "3")
+    (pin "2")
+    (instances
+      (project "01-getting-started"
+        (path "/8453acb3-9a68-4a83-979e-7b2f2c54f07b"
+          (reference "SW1") (unit 1)
+        )
+      )
+    )
+  )
+  (symbol (lib_id "power:PWR_FLAG") (at 119.38 72.39 90) (unit 1)
+    (in_bom yes) (on_board yes) (dnp no)
+    (property "Reference" "#FLG01" (at 117.475 72.39 0)
+      (effects (font (size 1.27 1.27)) hide)
+    )
+    (property "Value" "PWR_FLAG" (at 114.3 72.39 0)
       (effects (font (size 1.27 1.27)))
     )
-    (property "Footprint" "" (at 119.38 77.47 0)
+    (property "Footprint" "" (at 119.38 72.39 0)
       (effects (font (size 1.27 1.27)) hide)
     )
-    (property "Datasheet" "~" (at 119.38 77.47 0)
+    (property "Datasheet" "~" (at 119.38 72.39 0)
       (effects (font (size 1.27 1.27)) hide)
     )
@@
     )
   )
-  (symbol (lib_id "Device:Battery_Cell") (at 119.38 92.71 0) (unit 1)
+  (symbol (lib_id "Device:Battery_Cell") (at 119.38 96.52 0) (unit 1)
     (in_bom yes) (on_board yes) (dnp no) (fields_autoplaced)
-    (property "Reference" "BT1" (at 123.19 89.5985 0)
+    (property "Reference" "BT1" (at 123.19 93.4085 0)
       (effects (font (size 1.27 1.27)) (justify left))
     )
-    (property "Value" "3V" (at 123.19 92.1385 0)
+    (property "Value" "3V" (at 123.19 95.9485 0)
       (effects (font (size 1.27 1.27)) (justify left))
     )
-    (property "Footprint" "Battery:BatteryHolder_Keystone_1058_1x2032" (at 119.38 91.186 90)
+    (property "Footprint" "Battery:BatteryHolder_Keystone_1058_1x2032" (at 119.38 94.996 90)
       (effects (font (size 1.27 1.27)) hide)
     )
-    (property "Datasheet" "~" (at 119.38 91.186 90)
+    (property "Datasheet" "~" (at 119.38 94.996 90)
       (effects (font (size 1.27 1.27)) hide)
     )
