File: 02-a-send-off-board/rodney-beacon/rodney-beacon.kicad_sch (KiCad schematic)
At the start: 0 parts

Commit message: Add schematic to project
Parts:
- added C1, C2: 0.1uF, symbol Device:C_Polarized_US
- added C3: 100pF, symbol Device:C_Polarized_US
- added C4, C6: 0.01uF, symbol Device:C_Small
- added C5: 0.1uF, symbol Device:C_Small
- added R1: 15k, symbol Device:R
- added R2: 1.8k, symbol Device:R
- added U1: LM555xN, Package_DIP:DIP-8_W7.62mm, symbol Timer:LM555xN
- added U2, U3: 74LS93, symbol 74xx:74LS93
- added U4: L7805, Package_TO_SOT_THT:TO-220-3_Horizontal_TabDown, symbol Regulator_Linear:L7805
Connections:
- new net: U2.1 (CP1..3), U2.12 (Q0)
- new net: U2.11 (Q3), U3.14 (CP0)
- new net: U1.3 (Q), U2.14 (CP0)
- new net: U2.2 (R0(1)), U2.3 (R0(2))
- new net: C4.1, U1.5 (CV)
- new net: R1.2, R2.1, U1.7 (DIS)
- new net: C5.1, R2.2, U1.2 (TR), U1.6 (THR)
- new net: U3.1 (CP1..3), U3.12 (Q0)
- new net: U3.2 (R0(1)), U3.3 (R0(2))
- new net +12V: C1.1, U4.1 (IN)
- new net GND: C1.2, C2.2, C3.2, C4.2, C5.2, C6.2, U1.1 (GND), U2.10 (GND), U3.10 (GND), U4.2 (GND)
- new net power: C2.1, C3.1, C6.1, R1.1, U1.4 (R), U1.8 (VCC), U2.5 (VCC), U3.5 (VCC), U4.3 (OUT)

Commit message: Update design file
Parts:
- C1, C2, C3: footprint (none) -> Capacitor_SMD:CP_Elec_3x5.3
- C4, C5, C6: footprint (none) -> Capacitor_SMD:C_0201_0603Metric
- R1, R2: footprint (none) -> Resistor_SMD:R_0201_0603Metric
- U2, U3: footprint (none) -> Package_DIP:DIP-14_W7.62mm
Connections:
- net GND: no longer C6.2, U3.10 (GND)
- new net: C6.2, U3.10 (GND)
Changed lines of the file:
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@@
   (junction (at 86.36 127) (diameter 0) (color 0 0 0 0)
   )
-  (junction (at 196.85 127) (diameter 0) (color 0 0 0 0)
-  )
   (junction (at 156.21 62.23) (diameter 0) (color 0 0 0 0)
   )
   (junction (at 125.73 62.23) (diameter 0) (color 0 0 0 0)
   )
-  (junction (at 156.21 127) (diameter 0) (color 0 0 0 0)
-  )
   (junction (at 64.77 62.23) (diameter 0) (color 0 0 0 0)
   )
@@
   )
   (wire (pts (xy 120.65 87.63) (xy 125.73 87.63))
-    (stroke (width 0) (type default))
-  )
-  (wire (pts (xy 156.21 127) (xy 196.85 127))
     (stroke (width 0) (type default))
   )
@@
       (effects (font (size 1.27 1.27)) (justify left))
     )
-    (property "Footprint" "" (at 156.21 86.36 0)
+    (property "Footprint" "Package_DIP:DIP-14_W7.62mm" (at 156.21 86.36 0)
       (effects (font (size 1.27 1.27)) hide)
     )
@@
       (effects (font (size 1.27 1.27)) (justify left))
     )
-    (property "Footprint" "" (at 64.77 78.74 0)
+    (property "Footprint" "Capacitor_SMD:CP_Elec_3x5.3" (at 64.77 78.74 0)
       (effects (font (size 1.27 1.27)) hide)
     )
@@
       (effects (font (size 1.27 1.27)) (justify left))
     )
-    (property "Footprint" "" (at 86.36 120.65 0)
+    (property "Footprint" "Capacitor_SMD:C_0201_0603Metric" (at 86.36 120.65 0)
       (effects (font (size 1.27 1.27)) hide)
     )
@@
       (effects (font (size 1.27 1.27)) (justify left))
     )
-    (property "Footprint" "" (at 123.952 93.98 90)
+    (property "Footprint" "Resistor_SMD:R_0201_0603Metric" (at 123.952 93.98 90)
       (effects (font (size 1.27 1.27)) hide)
     )
@@
       (effects (font (size 1.27 1.27)) (justify left))
     )
-    (property "Footprint" "" (at 125.73 110.49 0)
+    (property "Footprint" "Capacitor_SMD:C_0201_0603Metric" (at 125.73 110.49 0)
       (effects (font (size 1.27 1.27)) hide)
     )
@@
       (effects (font (size 1.27 1.27)) (justify left))
     )
-    (property "Footprint" "" (at 196.85 86.36 0)
+    (property "Footprint" "Package_DIP:DIP-14_W7.62mm" (at 196.85 86.36 0)
       (effects (font (size 1.27 1.27)) hide)
     )
@@
       (effects (font (size 1.27 1.27)) (justify left))
     )
-    (property "Footprint" "" (at 76.2 95.25 0)
+    (property "Footprint" "Capacitor_SMD:CP_Elec_3x5.3" (at 76.2 95.25 0)
       (effects (font (size 1.27 1.27)) hide)
     )
@@
       (effects (font (size 1.27 1.27)) (justify left))
     )
-    (property "Footprint" "" (at 123.952 71.12 90)
+    (property "Footprint" "Resistor_SMD:R_0201_0603Metric" (at 123.952 71.12 90)
       (effects (font (size 1.27 1.27)) hide)
     )
@@
       (effects (font (size 1.27 1.27)) (justify left))
     )
-    (property "Footprint" "" (at 217.17 68.58 0)
+    (property "Footprint" "Capacitor_SMD:C_0201_0603Metric" (at 217.17 68.58 0)
       (effects (font (size 1.27 1.27)) hide)
     )
@@
       (effects (font (size 1.27 1.27)) (justify left))
     )
-    (property "Footprint" "" (at 30.48 106.68 0)
-      (effects (font (size 1.27 1.27)) hide)
-    )
+    (property "Footprint" "Capacitor_SMD:CP_Elec_3x5.3" (at 30.48 106.68 0)
+      (effects (font (size 1.27 1.27)) hide)
+    )
